File: KiCAD files/DST-2.kicad_sch (KiCad schematic)
At the start: 41 parts, among them J1 Barrel_Jack_MountingPin, J2 FTSW, J3 Power, J4 Pot_Dis, J5 Pot_Tone, J6 Pot_Vol, Q1 2N3904, Q2 2N3904, Q3 2N3904, U1 TL072

Commit message: Modified schematic and started a new PCB design
Parts:
- removed J1: Barrel_Jack_MountingPin, Connector_BarrelJack:BarrelJack_Kycon_KLDX-0202-xC_Horizontal, symbol Connector:Barrel_Jack_MountingPin
- removed J2: FTSW, Connector_JST:JST_XH_B4B-XH-A_1x04_P2.50mm_Vertical, symbol Connector:Conn_01x04_Socket
- removed J3: Power, Connector_JST:JST_XH_B2B-XH-A_1x02_P2.50mm_Vertical, symbol Connector:Conn_01x02_Socket
- added C13: 10µF, Capacitor_THT:C_Radial_D5.0mm_H11.0mm_P2.00mm, symbol Device:C
- added C14: 100nF, Capacitor_SMD:C_0603_1608Metric_Pad1.08x0.95mm_HandSolder, symbol Device:C
- added C15: 47uF, Capacitor_THT:C_Radial_D5.0mm_H11.0mm_P2.00mm, symbol Device:C
- added D4: LED, LED_THT:LED_D5.0mm, symbol Device:LED
- added J1: FTSW, Connector_PinHeader_2.54mm:PinHeader_1x04_P2.54mm_Vertical, symbol Connector:Conn_01x04_Socket
- added R17, R18: 10k, Resistor_SMD:R_0603_1608Metric_Pad0.98x0.95mm_HandSolder, symbol Device:R
- added R19: 1k, Resistor_SMD:R_0603_1608Metric_Pad0.98x0.95mm_HandSolder, symbol Device:R
- added TP1: INPUT, TestPoint:TestPoint_Pad_D1.0mm, symbol Connector:TestPoint
- added TP2: Q2 COLLECTOR, TestPoint:TestPoint_Pad_D1.0mm, symbol Connector:TestPoint
- added TP3: OP1 IN, TestPoint:TestPoint_Pad_D1.0mm, symbol Connector:TestPoint
- added TP4: OP1 OUT, TestPoint:TestPoint_Pad_D1.0mm, symbol Connector:TestPoint
- added TP5: OP-AMP OUTPUT, TestPoint:TestPoint_Pad_D1.0mm, symbol Connector:TestPoint
- added TP6: CLIPPING, TestPoint:TestPoint_Pad_D1.0mm, symbol Connector:TestPoint
- added TP7: Q3 B, TestPoint:TestPoint_Pad_D1.0mm, symbol Connector:TestPoint
- D1, D2, D3: footprint Diode_THT:D_DO-35_SOD27_P7.62mm_Horizontal -> Diode_SMD:D_SOD-323F
- J4, J5, J6: footprint Connector_JST:JST_XH_B3B-XH-A_1x03_P2.50mm_Vertical -> Connector_PinHeader_2.54mm:PinHeader_1x03_P2.54mm_Vertical
- Q1, Q2, Q3: footprint Package_TO_SOT_THT:TO-92_Inline -> Package_TO_SOT_SMD:TSOT-23_HandSoldering
- U1: footprint Package_DIP:DIP-8_W8.89mm_SMDSocket_LongPads -> Package_SO:SOIC-8_5.3x5.3mm_P1.27mm
Connections:
- net +4,5v: now also C13.1, R17.2, R18.1
- net +9V: now also C14.1, C15.1, D4.2 (A), J1.3 (Pin_3), R17.1
- net GND: now also C13.2, C14.2, C15.2, J1.4 (Pin_4), R18.2, R19.2
- net at U1.1, U1.2 (-), U1.5 (+): now also TP4.1
- net at C6.1, J4.1 (Pin_1), R11.1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: now also TP5.1
- net at C1.2, Q1.2 (B), R1.2: now also TP1.1
- net at C4.2, C5.1, Q2.3 (C)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: now also TP2.1
- net at D1.1 (K), R8.2, U1.3 (+): now also TP3.1
- net at C11.2, Q3.2 (B), R15.2: now also TP7.1
- net at C8.2, C9.1, D2.1 (K)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: now also TP6.1
- new net: D4.1 (K), R19.1
- new net IN_P: J1.1 (Pin_1)
- new net OUT_P: J1.2 (Pin_2)
Other:
- moved on the sheet: C1, C10, C11, C12, C2, C3, C4, C5, C6, C7, C8, C9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

Commit message: Finished PCB design
Connections:
- net in_p is gone; now on net IN_P: C1.1
- net out_p is gone; now on net OUT_P: C12.2
Changed lines of the file:
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@@
 		)
 	)
-	(global_label "in_p"
+	(global_label "IN_P"
 		(shape input)
 		(at 57.15 92.71 180)
@@
 		)
 		(property "Intersheetrefs" "${INTERSHEET_REFS}"
-			(at 50.2944 92.71 0)
+			(at 49.9919 92.71 0)
 			(hide yes)
 			(show_name no)
@@
 		)
 	)
-	(global_label "out_p"
+	(global_label "OUT_P"
 		(shape input)
 		(at 226.06 100.33 0)
@@
 		)
 		(property "Intersheetrefs" "${INTERSHEET_REFS}"
-			(at 234.1855 100.33 0)
+			(at 234.9114 100.33 0)
 			(hide yes)
 			(show_name no)
